Commit message: CartPole Notebook: Migrate to use mujoco to be able to visualize on Colab (#7)
* Request GPU on colab

* Workaround MuJoCo URDF parser bug

* Remove JAX installation and update `IS_COLAB` flag

---------

Co-authored-by: Filippo Luca Ferretti <102977828+flferretti@users.noreply.github.com>

File: examples/assets/cartpole.urdf (robot description, URDF)
Before this commit: robot cartpole, 4 links, 3 joints
Joints:
- joint pivot: limit lower=-3.4028234663852886e+38 upper=3.4028234663852886e+38 effort=500.0 velocity=10.0 -> lower=-100000000 upper=100000000 effort=500.0 velocity=10.0

Commit message: Update cartpole model and add missing script to generate it

File: examples/assets/cartpole.urdf (robot description, URDF)
Before this commit: robot cartpole, 4 links, 3 joints
Links:
- link pole: mass 0.1 -> 0.5
Joints:
- joint pivot: limit lower=-100000000 upper=100000000 effort=500.0 velocity=10.0 -> effort=3.4028235e+38 velocity=3.4028235e+38; type revolute -> continuous

Commit message: Update cartpole model in unit tests

File: examples/assets/cartpole.urdf (robot description, URDF)
Before this commit: robot cartpole, 4 links, 3 joints
Links:
- added link cart_frame
- added link rail_frame
Joints:
- added joint cart_frame_joint: type fixed, parent cart, child cart_frame, origin xyz=0.0 0.0 0.0 rpy=0.0 0.0 0.0
- added joint rail_frame_joint: type fixed, parent rail, child rail_frame, origin xyz=0.0 0.0 1.2 rpy=0.0 0.0 0.0
